File: PCB.C/REV.C.kicad_pcb (KiCad board)
At the start: 4 copper layers, 120 x 80 mm, 143 parts, among them J1 48204-0001, J2 GAMEPORT, J3 USB_HID, J4 VGA_IN, J5 MICRO_SD, J6 AUDIO_OUT, J7 Wuerth Elektronik 7499010211A, J8 POWER_IN, J9 WAVETABLE, P1 PWR_SW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

Commit message: 250527_1
cleaned up BOM
Parts:
- C13, C24, C40, C49: value 0.1uF -> 100nF
- C29: footprint SnipE Footprints:C_0805_2012Metric -> SnipE Footprints:C_1206_3216Metric
- C46, C5: value 33uF -> 47uF
- C47, C48: value 47uF -> 100uF
- FB1: value FB -> 600Ω@100MHz
- R19: value 33R -> 75
- R37: value 100R -> 150
- R42, R47: footprint Resistor_SMD:R_0603_1608Metric -> SnipE Footprints:R_0603_1608Metric
- moved C35 1.16 mm to (159.0, 78.7)
- moved C29 0.44 mm to (154.2, 78.7)
Routing:
- net +3.3V: track 199.8 -> 202.5 mm, vias 12 -> 16
- net /HSYNC: track 94.3 -> 93.0 mm, vias 2 -> 1
- net VCC: track 74.4 -> 75.5 mm
- net AGND: track 36.7 -> 36.0 mm
