File: PCB.C/REV.C.kicad_sch (KiCad schematic)
At the start: 142 parts, among them J1 48204-0001, J2 GAMEPORT, J3 USB_HID, J4 VGA_IN, J5 MICRO_SD, J6 AUDIO_OUT, J7 Wuerth Elektronik 7499010211A, J8 POWER_IN, J9 WAVETABLE, P1 PWR_SW, Q1 Q_PMOS_GDS, Q2 NPN, SW2 RESET, SW3 HID_PRG, U1 SOM304RD-VI, U2 U_K24C08, U3 CS4237B-KQ, U4 AMS1117-3.3, U5 U_MAX16054, U6 CH559L, U7 74LVC2G07, X1 16.9344MHz, X2 12MHz

Commit message: 250527_1
cleaned up BOM
Parts:
- BT1: symbol llama_shared:BT -> SnipE Symbol Library:BT; LCSC C964745 -> (none); Label CR1220 -> (none); Part Number (none) -> LCSC:C964818
- C1, C2, C3, C37, C4, C44, C45, C51, C7, C8: symbol llama_shared:C -> SnipE Symbol Library:C; LCSC C1525 -> (none); Note Hold@1A -> (none); Note2 Trip@1.8A -> (none); Part Number (none) -> DIGIKEY:C0603C104K3RACTU
- C10, C9: symbol llama_shared:C -> SnipE Symbol Library:C; LCSC C76960 -> (none); Note Hold@1A -> (none); Note2 Trip@1.8A -> (none); Part Number (none) -> DIGIKEY:C0603C220J8GACTU
- C11, C12: symbol llama_shared:C -> SnipE Symbol Library:C; LCSC C76947 -> (none); Note C0G -> (none); Note2 Trip@1.8A -> (none); Part Number (none) -> DIGIKEY:GRM1885C1H102JA01D
- C13, C24, C40: value 0.1uF -> 100nF; symbol llama_shared:C -> SnipE Symbol Library:C; LCSC C207017 -> (none); Note Hold@1A -> (none); Note2 Trip@1.8A -> (none); Part Number (none) -> DIGIKEY:C0603C104K3RACTU
- C14, C17, C18, C19: symbol Device:C_Small -> SnipE Symbol Library:C_Small; LCSC C207017 -> (none); Note Hold@1A -> (none); Note2 Trip@1.8A -> (none); Part Number (none) -> DIGIKEY:C0603C102K3RACTU
- C15, C16: symbol llama_shared:C -> SnipE Symbol Library:C; LCSC C207017 -> (none); Note Hold@1A -> (none); Note2 Trip@1.8A -> (none); Part Number (none) -> DIGIKEY:C0603C106M9PACTU
- C20, C21, C22, C23: symbol Device:C_Small -> SnipE Symbol Library:C_Small; LCSC C207017 -> (none); Note Hold@1A -> (none); Note2 Trip@1.8A -> (none); Part Number (none) -> DIGIKEY:C0603C562K3RACTU
- C25: symbol llama_shared:C -> SnipE Symbol Library:C; Part Number (none) -> DIGIKEY:GRM31CR61A107MEA8K
- C26: symbol llama_shared:C -> SnipE Symbol Library:C; LCSC C14663 -> (none); Note Hold@1A -> (none); Note2 Trip@1.8A -> (none); Part Number (none) -> DIGIKEY:C0603C104K3RACTU
- C27, C28: symbol llama_shared:C -> SnipE Symbol Library:C; LCSC C207017 -> (none); Note C0G -> (none); Note2 Trip@1.8A -> (none); Part Number (none) -> DIGIKEY:GRM1885C1H102JA01D
- C29: footprint SnipE Footprints:C_0805_2012Metric -> SnipE Footprints:C_1206_3216Metric; symbol llama_shared:C -> SnipE Symbol Library:C; Part Number (none) -> DIGIKEY:C1206C106K4PACTU
- C30: symbol llamablaster:C -> SnipE Symbol Library:C; LCSC C1525 -> (none); Note Hold@1A -> (none); Note2 Trip@1.8A -> (none); Part Number (none) -> DIGIKEY:C0603C104K3RACTU
- C31: symbol llama_shared:C -> SnipE Symbol Library:C; LCSC C207017 -> (none); Note Hold@1A -> (none); Note2 Trip@1.8A -> (none); Part Number (none) -> DIGIKEY:C0603C272K5RACTU
- C32, C33, C34, C36: symbol Device:C_Small -> SnipE Symbol Library:C_Small; LCSC C207017 -> (none); Note Hold@1A -> (none); Note2 Trip@1.8A -> (none); Part Number (none) -> DIGIKEY:C0603C104K3RACTU
- C35, C41: symbol llama_shared:C -> SnipE Symbol Library:C; Part Number (none) -> DIGIKEY:C1206C476M8PACTU
- C38, C39: symbol llama_shared:C -> SnipE Symbol Library:C; Part Number (none) -> DIGIKEY: C1206C106K4PACTU
- C43: symbol llama_shared:C -> SnipE Symbol Library:C; LCSC C60133 -> (none); Note Hold@1A -> (none); Note2 Trip@1.8A -> (none); Part Number (none) -> DIGIKEY:C0603C103K5RACTU
- C46, C5: value 33uF -> 47uF; Part Number (none) -> DIGIKEY:C1206C476M8PACTU
- C47, C48: value 47uF -> 100uF; symbol llama_shared:C -> SnipE Symbol Library:C; Part Number (none) -> DIGIKEY:GRM31CR61A107MEA8K
- C49: value 0.1uF -> 100nF; symbol llama_shared:C -> SnipE Symbol Library:C; LCSC C14663 -> (none); Note Hold@1A -> (none); Note2 Trip@1.8A -> (none); Part Number (none) -> DIGIKEY:C0603C104K3RACTU
- C50: symbol llama_shared:C -> SnipE Symbol Library:C; LCSC C207017 -> (none); Note Hold@1A -> (none); Note2 Trip@1.8A -> (none); Part Number (none) -> DIGIKEY:C0603C335M9PACTU
- C52, C54: symbol llamablaster:C -> SnipE Symbol Library:C; LCSC C1663 -> (none); Note Hold@1A -> (none); Note2 Trip@1.8A -> (none); Part Number (none) -> LCSC:C1663
- C53: symbol llama_shared:C -> SnipE Symbol Library:C; LCSC C76947 -> (none); Part Number (none) -> DIGIKEY:C0603C102K5RACTU
- C6: symbol llama_shared:C -> SnipE Symbol Library:C; Part Number (none) -> DIGIKEY:C1206C105K3RACTU
- C61, C62: symbol llama_shared:C -> SnipE Symbol Library:C; LCSC C77009 -> (none); Part Number (none) -> DIGIKEY:C1206C105K3RACTU
- D1: LCSC C130723 -> (none); MANUFACTURER Lite-On Inc. -> (none); MAXIMUM_PACKAGE_HEIGHT 1mm -> (none); PARTREV D -> (none); Part Number (none) -> DIGIKEY:LTST-S220KGKT; STANDARD Manufacturer Recommendations -> (none)
- D2: LCSC C130723 -> (none); Label PWR_ON -> (none); MANUFACTURER Lite-On Inc. -> (none); MAXIMUM_PACKAGE_HEIGHT 1mm -> (none); PARTREV D -> (none); Part Number (none) -> DIGIKEY:LTST-S220KGKT; STANDARD Manufacturer Recommendations -> (none)
- D3: symbol llama_shared:D -> SnipE Symbol Library:D; LCSC C2128 -> (none); Part Number (none) -> DIGIKEY:1N4148WS-7-F
- F1, F2, F3, F4: symbol llama_shared:F -> SnipE Symbol Library:F; Part Number (none) -> DIGIKEY:0603L100SLYR
- FB1: value FB -> 600Ω@100MHz; symbol Device:FerriteBead -> SnipE Symbol Library:FerriteBead_Small; Note 600Ω@100MHz -> (none); Part Number (none) -> DIGIKEY:MPZ2012S601ATD25
- FB2: symbol Device:FerriteBead_Small -> SnipE Symbol Library:FerriteBead_Small; LCSC C160977 -> (none); Part Number (none) -> DIGIKEY:MPZ2012S601ATD25
- FB3, FB4: symbol Device:FerriteBead_Small -> SnipE Symbol Library:FerriteBead_Small; LCSC C107332 -> (none); Part Number (none) -> DIGIKEY:MPZ2012S101AT000
- J1: symbol weeCee_library:48204-0001 -> SnipE Symbol Library:48204-0001; Manufacturer_Name Molex -> (none); Manufacturer_Part_Number 48204-0001 -> (none); Mouser Part Number 538-48204-0001 -> (none); Mouser Price/Stock https://www.mouser.co.uk/ProductDetail/Molex/48204-0001?qs=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 -> (none); Part Number (none) -> DIGIKEY:0482040001
- J2: symbol llama_shared:J_DA15_Gameport -> SnipE Symbol Library:J_DA15_Gameport; LCSC C77835 -> (none); Part Number (none) -> LCSC:C77835
- J3: symbol llama_shared:J_USB_A_Stacked_C12049 -> SnipE Symbol Library:J_USB_A_Stacked_C12049; Part Number (none) -> DIGIKEY:C12049
- J4: symbol weeCee_library:634-015-263-032 -> SnipE Symbol Library:634-015-263-032; Height 12.93 -> (none); Manufacturer_Name EDAC -> (none); Manufacturer_Part_Number 634-015-263-032 -> (none); Mouser Part Number 587-634-015-263-032 -> (none); Mouser Price/Stock https://www.mouser.co.uk/ProductDetail/EDAC/634-015-263-032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 -> (none); Part Number (none) -> DIGIKEY:634-015-263-032
- J5: symbol llama_shared:J_Micro_SD_TF01A -> SnipE Symbol Library:J_Micro_SD_TF01A; LCSC C91145 -> (none); Part Number (none) -> LCSC:C91145
- J6: symbol Connector_Audio:AudioJack3 -> SnipE Symbol Library:AudioJack3
- J7: symbol llama_shared:7499010211A -> SnipE Symbol Library:7499010211A; Availability In Stock -> (none); Check_prices https://www.snapeda.com/parts/7499010211A/Wurth+Elektronik/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 -> (none); Description_1 10/100BASE-TX, THT, 1x1, Tab-down, without shield tabs, LED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 -> (none); MF Wurth Elektronik -> (none); MP 7499010211A -> (none); Package None -> (none); Part Number (none) -> DIGIKEY:7499010211A; Price None -> (none); Purchase-URL https://www.snapeda.com/api/url_track_click_mouser/?unipart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 -> (none); SnapEDA_Link https://www.snapeda.com/parts/7499010211A/Wurth+Elektronik/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 -> (none)
- J8: symbol llama_shared:J_USB_C -> SnipE Symbol Library:J_USB_C; Part Number (none) -> LCSC:C165948
- J9: symbol llama_shared:J_WAVETABLE -> SnipE Symbol Library:J_WAVETABLE; LCSC C2884022 -> (none); Part Number (none) -> LCSC:C2884022
- JP2: symbol Jumper:Jumper_2_Bridged -> SnipE Symbol Library:Jumper_2_Bridged; now left out of the parts list
- L1, L2, L3: symbol llama_shared:L_EMI_FILTER -> SnipE Symbol Library:L_EMI_FILTER; LCSC C315725 -> (none); Part Number (none) -> DIGIKEY:MCM2012B900GBEDG
- P1: Part Number (none) -> ALIEXPRESS
- Q1: symbol llama_shared:Q_PMOS_GDS -> SnipE Symbol Library:Q_PMOS_GDS; Part Number (none) -> DIGIKEY:DMP3099L-7
- Q2: symbol llama_shared:Q_NPN_BEC -> SnipE Symbol Library:Q_NPN_BEC; LCSC C2146 -> (none); Part Number (none) -> LCSC:C2146
- R1, R2, R3, R4, R5: symbol Device:R_Small -> SnipE Symbol Library:R_Small; LCSC C207017 -> (none); Note Hold@1A -> (none); Note2 Trip@1.8A -> (none); Part Number (none) -> DIGIKEY:RC0603FR-074K7L
- R10, R20, R43, R44, R45, R46, R9: symbol llama_shared:R -> SnipE Symbol Library:R; LCSC C207017 -> (none); Note Hold@1A -> (none); Note2 Trip@1.8A -> (none); Part Number (none) -> DIGIKEY:RC0603FR-074K7L
- R11, R6, R7, R8: symbol Device:R_Small -> SnipE Symbol Library:R_Small; LCSC C207017 -> (none); Note Hold@1A -> (none); Note2 Trip@1.8A -> (none); Part Number (none) -> DIGIKEY:RC0603FR-072K2L
- R12, R13, R14, R15, R16, R17: symbol Device:R_Small -> SnipE Symbol Library:R_Small; LCSC C207017 -> (none); Note Hold@1A -> (none); Note2 Trip@1.8A -> (none); Part Number (none) -> DIGIKEY:RC0603FR-0747KL
- R18, R28, R29, R30, R31, R32: symbol Device:R_Small -> SnipE Symbol Library:R_Small; LCSC C207017 -> (none); Note Hold@1A -> (none); Note2 Trip@1.8A -> (none); Part Number (none) -> DIGIKEY:RC0603JR-0733RL
- R19: value 33R -> 75; symbol tinyllama:R -> SnipE Symbol Library:R; LCSC C25867 -> (none); Note Hold@1A -> (none); Note2 Trip@1.8A -> (none); Part Number (none) -> DIGIKEY:RC0603JR-0775RL
- R21, R41: symbol llama_shared:R -> SnipE Symbol Library:R; LCSC C207017 -> (none); Note Hold@1A -> (none); Note2 Trip@1.8A -> (none); Part Number (none) -> DIGIKEY:RC0603FR-0747KL
- R22, R23, R24, R25: symbol Device:R_Small -> SnipE Symbol Library:R_Small; LCSC C207017 -> (none); Note Hold@1A -> (none); Note2 Trip@1.8A -> (none); Part Number (none) -> DIGIKEY:RC0603FR-0749R9L
- R26, R27: symbol Device:R_Small -> SnipE Symbol Library:R_Small; LCSC C207017 -> (none); Note Hold@1A -> (none); Note2 Trip@1.8A -> (none); Part Number (none) -> DIGIKEY:RC0603FR-071KL
- R33, R34, R35, R36: symbol llama_shared:R -> SnipE Symbol Library:R; LCSC C207017 -> (none); Note Hold@1A -> (none); Note2 Trip@1.8A -> (none); Part Number (none) -> DIGIKEY:RC0603JR-076K8L
- R37: value 100R -> 150; Indicator + -> (none); LCSC C207017 -> (none); Note Hold@1A -> (none); Note2 Trip@1.8A -> (none); Part Number (none) -> DIGIKEY:RC0603FR-07150RL; Rating W -> (none)
- R38: symbol llama_shared:R -> SnipE Symbol Library:R; LCSC C11702 -> (none); Note Hold@1A -> (none); Note2 Trip@1.8A -> (none); Part Number (none) -> DIGIKEY:RC0603FR-071KL
- R39, R40: symbol llama_shared:R -> SnipE Symbol Library:R; LCSC C207017 -> (none); Note Hold@1A -> (none); Note2 Trip@1.8A -> (none); Part Number (none) -> DIGIKEY:RC0603FR-075K1L
- R42: footprint Resistor_SMD:R_0603_1608Metric -> SnipE Footprints:R_0603_1608Metric; symbol llama_shared:R -> SnipE Symbol Library:R; Part Number (none) -> DIGIKEY:RC0603FR-0710KL
- R47: footprint Resistor_SMD:R_0603_1608Metric -> SnipE Footprints:R_0603_1608Metric; symbol llama_shared:R -> SnipE Symbol Library:R; Part Number (none) -> DIGIKEY:RC0603JR-07470RL
- SP1: LCSC C252917 -> (none); Label PC SPEAKER -> (none); MANUFACTURER Pui Audio -> (none); MAXIMUM_PACKAGE_HEIGHT 4.2 mm -> (none); PARTREV 1/19/2017 -> (none); Part Number (none) -> DIGIKEY:SP3243EEA-L/TR; STANDARD Manufacturer Recommendations -> (none)
- SW2: LCSC C5342982 -> (none); Label PWR -> (none); MANUFACTURER TE Connectivity -> (none); PARTREV G4 -> (none); Part Number (none) -> LCSC:C2859426; STANDARD Manufacturer Recommednation -> (none)
- SW3: LCSC C5342982 -> (none); Label HID_PRG -> (none); MANUFACTURER TE Connectivity -> (none); PARTREV G4 -> (none); Part Number (none) -> LCSC:C2859426; STANDARD Manufacturer Recommednation -> (none)
- U1: symbol weeCee_library:SOM304RD-VI -> SnipE Symbol Library:SOM304RD-VI; Part Number (none) -> ICOP
- U2: symbol llama_shared:U_K24C08 -> SnipE Symbol Library:U_K24C08; Part Number (none) -> DIGIKEY:24LC08BT-I/OT
- U3: Part Number (none) -> UTSOURCE
- U4: symbol llama_shared:U_AMS1117-3.3 -> SnipE Symbol Library:U_AMS1117-3.3; Part Number (none) -> DIGIKEY:AMS1117-3.3
- U5: symbol llama_shared:U_MAX16054 -> SnipE Symbol Library:U_MAX16054; Part Number (none) -> DIGIKEY:MAX16054AZT+T
- U6: symbol tinyllama:U_CH559L -> SnipE Symbol Library:U_CH559L; LCSC C150548 -> (none)
- U7: symbol tinyllama:U_74LVC2G07 -> SnipE Symbol Library:U_74LVC2G07; LCSC C7849 -> (none); Part Number (none) -> DIGIKEY:SN74LVC2G07DCKR
- X1: symbol llama_shared:X -> SnipE Symbol Library:X; LCSC C4944017 -> (none); Part Number (none) -> LCSC:C4944017
- X2: symbol tinyllama:X_GND24 -> SnipE Symbol Library:X_GND24; LCSC C9002 -> (none); Part Number (none) -> LCSC:C9002
Other:
- note removed: "ORANGE"
- moved on the sheet: C27, C28, C29, C35, C38, C39, C49, U4
